File: CAD/shield.kicad_pcb (KiCad board)
At the start: 2 copper layers, 91.4 x 59.7 mm, 21 parts, among them J1 Reg 3, J10 Power, J11 Analog 1, J12 Analog 2, J13 Digital 3, J14 Comm, J15 Digital 1, J16 Digital 2, J17 Analog 2, J18 Analog 1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

Commit message: updated schematic
Parts:
- added J22: Calcant, Connector_PinHeader_2.54mm:PinHeader_1x03_P2.54mm_Vertical, F.Cu at (219.6, 91.3)
- moved J16 22.9 mm to (157.5, 66.0), turned to 90 degrees
- moved J3 22.9 mm to (157.5, 69.8), turned to -90 degrees
- moved J15 17.8 mm to (180.3, 66.0), turned to 90 degrees
- moved J4 17.8 mm to (180.3, 69.8), turned to -90 degrees
- moved J8 2.54 mm to (160.0, 109.2)
Connections:
- J13 pad 15: unconnected-(J13-Pin_15-Pad15) -> Net-(J13-Pin_15)
- J13 pad 17: unconnected-(J13-Pin_17-Pad17) -> Net-(J13-Pin_17)
- J15 pad 1: Net-(J15-Pin_1) -> unconnected-(J15-Pin_1-Pad1)
- J15 pad 2: Net-(J15-Pin_2) -> unconnected-(J15-Pin_2-Pad2)
- J15 pad 7: unconnected-(J15-Pin_7-Pad7) -> Net-(J15-Pin_7)
- J15 pad 8: unconnected-(J15-Pin_8-Pad8) -> Net-(J15-Pin_8)
- J4 pad 1: Net-(J15-Pin_1) -> Net-(J15-Pin_3)
- J4 pad 2: Net-(J15-Pin_2) -> Net-(J15-Pin_4)
- J4 pad 3: Net-(J15-Pin_3) -> Net-(J15-Pin_5)
- J4 pad 4: Net-(J15-Pin_4) -> Net-(J15-Pin_6)
- J4 pad 5: Net-(J15-Pin_5) -> Net-(J15-Pin_7)
- J4 pad 6: Net-(J15-Pin_6) -> Net-(J15-Pin_8)
Routing:
- net +5VD: track 56.9 -> 44.3 mm
- net Net-(J13-Pin_15): track 0.00 -> 12.3 mm
- net Net-(J13-Pin_17): track 0.00 -> 10.8 mm
- net GND: track 141.2 -> 151.6 mm
- net Net-(J15-Pin_7): track 0.00 -> 7.25 mm
- net Net-(J15-Pin_8): track 0.00 -> 6.66 mm
- net Net-(J15-Pin_2): track 3.81 -> 0.00 mm
- net Net-(J15-Pin_1): track 3.81 -> 0.00 mm
- net Net-(J15-Pin_4): track 3.81 -> 7.55 mm
- net Net-(J15-Pin_3): track 3.81 -> 7.55 mm
- net Net-(J15-Pin_5): track 3.81 -> 7.10 mm
- net Net-(J15-Pin_6): track 3.81 -> 6.66 mm
- net Net-(J19-Pin_8): track 7.62 -> 5.08 mm
- net Net-(J19-Pin_7): track 7.62 -> 5.08 mm
