File: CAD/shield.kicad_sch (KiCad schematic)
At the start: 21 parts, among them J1 Reg 3, J10 Power, J11 Analog 1, J12 Analog 2, J13 Digital 3, J14 Comm, J15 Digital 1, J16 Digital 2, J17 Analog 2, J18 Analog 1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

Commit message: updated schematic
Parts:
- added J22: Calcant, Connector_PinHeader_2.54mm:PinHeader_1x03_P2.54mm_Vertical, symbol Connector:Conn_01x03_Pin
Connections:
- net GND: now also J22.3 (Pin_3)
- net at J4.1 (Pin_1): now also J15.3 (Pin_3); no longer J15.1 (Pin_1)
- net at J4.2 (Pin_2): now also J15.4 (Pin_4); no longer J15.2 (Pin_2)
- net at J4.3 (Pin_3): now also J15.5 (Pin_5); no longer J15.3 (Pin_3)
- net at J4.4 (Pin_4): now also J15.6 (Pin_6); no longer J15.4 (Pin_4)
- net at J4.5 (Pin_5): now also J15.7 (Pin_7); no longer J15.5 (Pin_5)
- net at J4.6 (Pin_6): now also J15.8 (Pin_8); no longer J15.6 (Pin_6)
- net at J13.15 (Pin_15): now also J22.1 (Pin_1)
- net at J13.17 (Pin_17): now also J22.2 (Pin_2)
Other:
- moved on the sheet: J10, J11, J12, J14, J15, J16, J17, J18, J19, J2, J20, J21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
