File: CAD/Stops/Stops.kicad_pcb (KiCad board)
At the start: 2 copper layers, 60 x 33 mm, 11 parts, among them J1 Conn_01x08_Socket, SW1 SW_Push_LED, SW2 SW_Push_LED, SW3 SW_Push_LED

Commit message: redo CAD
Parts:
- J1: footprint Connector_PinHeader_2.54mm:PinHeader_1x08_P2.54mm_Horizontal -> Connector_IDC:IDC-Header_2x05_P2.54mm_Latch_Horizontal; moved to B.Cu
- moved R3 32.1 mm to (84.8, 63.0)
- moved SW3 32.1 mm to (88.2, 52.2)
- moved R1 32.1 mm to (116.9, 63.0)
- moved SW1 32.1 mm to (120.4, 52.2)
- moved J1 11.7 mm to (109.5, 41.5)
Connections:
- net Net-(J1-Pin_1) renamed /SW1
- net Net-(J1-Pin_2) renamed /L1
- net Net-(J1-Pin_3) renamed /SW2
- net Net-(J1-Pin_4) renamed /L2
- net Net-(J1-Pin_5) renamed /SW3
- net Net-(J1-Pin_6) renamed /L3
- J1 pad 7: GND -> unconnected-(J1-Pin_7-Pad7)
- J1 pad 8: GND -> unconnected-(J1-Pin_8-Pad8)
Routing:
- net /L1: track 17.7 -> 28.1 mm
- net /SW3: track 26.3 -> 22.7 mm
- net GND: track 85.9 -> 89.5 mm
- net /SW1: track 20.0 -> 22.9 mm
- net /L3: track 24.2 -> 22.6 mm
- net /L2: track 17.2 -> 18.7 mm
- net /SW2: track 18.2 -> 16.8 mm
