File: CAD/Stops/Stops.kicad_sch (KiCad schematic)
At the start: 11 parts, among them J1 Conn_01x08_Socket, SW1 SW_Push_LED, SW2 SW_Push_LED, SW3 SW_Push_LED

Commit message: save
Parts:
- H1: renamed from H3; KiLib_Generator (none) -> mounting_hardware/mounting_hole
- H2: renamed from H1; KiLib_Generator (none) -> mounting_hardware/mounting_hole
- H3: renamed from H4; KiLib_Generator (none) -> mounting_hardware/mounting_hole
- H4: renamed from H2; KiLib_Generator (none) -> mounting_hardware/mounting_hole
- J1: KiLib_Generator (none) -> connector/pin_header_socket
- R1: renamed from R2; KiLib_Generator (none) -> resistor/THT
- R2: renamed from R1; KiLib_Generator (none) -> resistor/THT
- R3: KiLib_Generator (none) -> resistor/THT
- renumbered SW2 to SW1, SW1 to SW2
Changed lines of the file:
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@@
 		(dnp no)
 		(fields_autoplaced yes)
-		(property "Reference" "SW1"
+		(property "Reference" "SW2"
 			(at 80.01 50.8 0)
 			(show_name no)
@@
 			(project "Stops"
 				(path "/8700c023-aa1e-4c84-a44d-574e616a3737"
-					(reference "SW1")
+					(reference "SW2")
 					(unit 1)
 				)
@@
 			)
 		)
+		(property "KiLib_Generator" "connector/pin_header_socket"
+			(at 113.03 52.07 0)
+			(hide yes)
+			(show_name no)
+			(do_not_autoplace no)
+			(effects
+				(font
+					(size 1.27 1.27)
+				)
+			)
+		)
 		(pin "6"
 		)
@@
 		(in_pos_files yes)
 		(dnp no)
-		(property "Reference" "R2"
+		(property "Reference" "R1"
 			(at 66.548 48.006 90)
 			(show_name no)
@@
 			)
 		)
+		(property "KiLib_Generator" "resistor/THT"
+			(at 68.58 45.72 0)
+			(hide yes)
+			(show_name no)
+			(do_not_autoplace no)
+			(effects
+				(font
+					(size 1.27 1.27)
+				)
+			)
+		)
 		(pin "2"
 		)
@@
 			(project "Stops"
 				(path "/8700c023-aa1e-4c84-a44d-574e616a3737"
-					(reference "R2")
+					(reference "R1")
 					(unit 1)
 				)
@@
 		(dnp no)
 		(fields_autoplaced yes)
-		(property "Reference" "H1"
+		(property "Reference" "H2"
 			(at 102.87 30.4799 0)
 			(show_name no)
@@
 			)
 		)
-		(instances
-			(project "Stops"
-				(path "/8700c023-aa1e-4c84-a44d-574e616a3737"
-					(reference "H1")
+		(property "KiLib_Generator" "mounting_hardware/mounting_hole"
+			(at 100.33 31.75 0)
+			(hide yes)
+			(show_name no)
+			(do_not_autoplace no)
+			(effects
+				(font
+					(size 1.27 1.27)
+				)
+			)
+		)
+		(instances
+			(project "Stops"
+				(path "/8700c023-aa1e-4c84-a44d-574e616a3737"
+					(reference "H2")
 					(unit 1)
 				)
@@
 		(dnp no)
 		(fields_autoplaced yes)
-		(property "Reference" "H2"
+		(property "Reference" "H4"
 			(at 120.65 30.4799 0)
 			(show_name no)
@@
 			)
 		)
-		(instances
-			(project "Stops"
-				(path "/8700c023-aa1e-4c84-a44d-574e616a3737"
-					(reference "H2")
+		(property "KiLib_Generator" "mounting_hardware/mounting_hole"
+			(at 118.11 31.75 0)
+			(hide yes)
+			(show_name no)
+			(do_not_autoplace no)
+			(effects
+				(font
+					(size 1.27 1.27)
+				)
+			)
+		)
+		(instances
+			(project "Stops"
+				(path "/8700c023-aa1e-4c84-a44d-574e616a3737"
+					(reference "H4")
 					(unit 1)
 				)
@@
 		(dnp no)
 		(fields_autoplaced yes)
-		(property "Reference" "H4"
+		(property "Reference" "H3"
 			(at 157.48 30.4799 0)
 			(show_name no)
@@
 			)
 		)
-		(instances
-			(project "Stops"
-				(path "/8700c023-aa1e-4c84-a44d-574e616a3737"
-					(reference "H4")
+		(property "KiLib_Generator" "mounting_hardware/mounting_hole"
+			(at 154.94 31.75 0)
+			(hide yes)
+			(show_name no)
+			(do_not_autoplace no)
+			(effects
+				(font
+					(size 1.27 1.27)
+				)
+			)
+		)
+		(instances
+			(project "Stops"
+				(path "/8700c023-aa1e-4c84-a44d-574e616a3737"
+					(reference "H3")
 					(unit 1)
 				)
@@
 			)
 		)
+		(property "KiLib_Generator" "resistor/THT"
+			(at 68.58 77.47 0)
+			(hide yes)
+			(show_name no)
+			(do_not_autoplace no)
+			(effects
+				(font
+					(size 1.27 1.27)
+				)
+			)
+		)
 		(pin "2"
 		)
@@
 		(dnp no)
 		(fields_autoplaced yes)
-		(property "Reference" "SW2"
+		(property "Reference" "SW1"
 			(at 80.01 35.56 0)
 			(show_name no)
@@
 			(project "Stops"
 				(path "/8700c023-aa1e-4c84-a44d-574e616a3737"
-					(reference "SW2")
+					(reference "SW1")
 					(unit 1)
 				)
@@
 		(in_pos_files yes)
 		(dnp no)
-		(property "Reference" "R1"
+		(property "Reference" "R2"
 			(at 66.548 63.246 90)
 			(show_name no)
@@
 			)
 		)
+		(property "KiLib_Generator" "resistor/THT"
+			(at 68.58 60.96 0)
+			(hide yes)
+			(show_name no)
+			(do_not_autoplace no)
+			(effects
+				(font
+					(size 1.27 1.27)
+				)
+			)
+		)
 		(pin "2"
 		)
@@
 			(project "Stops"
 				(path "/8700c023-aa1e-4c84-a44d-574e616a3737"
-					(reference "R1")
+					(reference "R2")
 					(unit 1)
 				)
@@
 		(dnp no)
 		(fields_autoplaced yes)
-		(property "Reference" "H3"
+		(property "Reference" "H1"
 			(at 139.7 30.4799 0)
 			(show_name no)
@@
 			)
 		)
-		(instances
-			(project "Stops"
-				(path "/8700c023-aa1e-4c84-a44d-574e616a3737"
-					(reference "H3")
-					(unit 1)
-				)
+		(property "KiLib_Generator" "mounting_hardware/mounting_hole"
+			(at 137.16 31.75 0)
+			(hide yes)
+			(show_name no)
+			(do_not_autoplace no)
+			(effects
+				(font
+					(size 1.27 1.27)
+				)
+			)
+		)
+		(instances
+			(project "Stops"
+				(path "/8700c023-aa1e-4c84-a44d-574e616a3737"
+					(reference "H1")
+					(unit 1)
+				)

Commit message: redo CAD
Parts:
- J1: footprint Connector_PinHeader_2.54mm:PinHeader_1x08_P2.54mm_Horizontal -> Connector_IDC:IDC-Header_2x05_P2.54mm_Latch_Horizontal; symbol Connector:Conn_01x08_Socket -> Connector_Generic:Conn_02x05_Odd_Even
Connections:
- net GND: now also J1.10 (Pin_10), J1.9 (Pin_9); no longer J1.7 (Pin_7), J1.8 (Pin_8)
- net L2: now reaches J1.3 (Pin_3)
- net L2: now also SW2.4 (A); no longer SW2.2
- net SW2: now reaches J1.4 (Pin_4)
- net SW2: now also SW2.2; no longer SW2.4 (A)
- net L1: now reaches J1.1 (Pin_1)
- net L1: now also SW1.4 (A); no longer SW1.2
- net SW1: now reaches J1.2 (Pin_2)
- net SW1: now also SW1.2; no longer SW1.4 (A)
- net L3: now reaches J1.5 (Pin_5)
- net L3: now also SW3.4 (A); no longer SW3.2
- net SW3: now reaches J1.6 (Pin_6)
- net SW3: now also SW3.2; no longer SW3.4 (A)
Other:
- moved on the sheet: J1
